File: hardware/myproject.kicad_pcb (KiCad board)
At the start: 2 copper layers, 0 parts

Commit message: updated README.md & added OHL texts
Other:
- board text added: "Licensed under CERN OHL v.1.2"
Changed lines of the file:
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@@
     (area 0 0 0 0)
     (thickness 1.6)
-    (drawings 0)
+    (drawings 1)
     (tracks 0)
     (zones 0)
@@
     (uvia_drill 0.1)
   )
+  (gr_text "Licensed under CERN OHL v.1.2" (at 143.9164 63.8302) (layer F.SilkS)
+    (effects (font (size 1 1) (thickness 0.125)))
+  )
 )
