File: hardware/myproject.sch (KiCad schematic (older format))
At the start: 0 parts

Commit message: updated README.md & added OHL texts
Other:
- note added: "Licensed under CERN OHL v.1.2"
Changed lines of the file:
@@
 LIBS:contrib
 LIBS:valves
+LIBS:myproject-cache
 EELAYER 25 0
 EELAYER END
@@
 Comment4 ""
 $EndDescr
+Text Notes 600  7675 0    118  ~ 0
+Licensed under CERN OHL v.1.2
 $EndSCHEMATC
